Commit message: Agrega inercias, colisiones y plugins al URDF

File: src/robot_description/urdf/colmibot.urdf (robot description, URDF)
Before this commit: robot colmibot, 8 links, 7 joints
Links:
- link camara_link: mass None -> 0.3018622
- link chasis_link: mass None -> 1.8203639
- link imu_link: mass None -> 0.003012336
- link rueda_derecha_link: mass None -> 0.019358118; geometry collision cylinder length=0.012 radius=0.030; visual mesh filename=package://robot_description/meshes/rueda_derecha.stl
- link rueda_izquierda_link: mass None -> 0.019358118; geometry collision cylinder length=0.012 radius=0.030; visual mesh filename=package://robot_description/meshes/rueda_izquierda.stl
- link rueda_loca_link: mass None -> 0.12378384; geometry collision sphere radius=0.0135; collision sphere radius=0.0135
- link tof_link: mass None -> 0.017814617
